File: PCB/Synth_arduino_nano.kicad_pcb (KiCad board)
At the start: 2 copper layers, 15 parts, among them J1 FSLP, J3 Encoder, U1 DM-OLED096-636

Commit message: Add files via upload
Parts:
- removed J3: Encoder, Connector_PinSocket_2.54mm:PinSocket_1x05_P2.54mm_Horizontal
- added R4: VibratoIntensity, PTV09A:PTV09A-4025F-B103, F.Cu at (119.4, 83.8)
- added R5: VibratoFrequency, PTV09A:PTV09A-4025F-B103, F.Cu at (134.6, 83.8)
- added R6: 10k, Resistor_SMD:R_0805_2012Metric_Pad1.20x1.40mm_HandSolder, F.Cu at (99.0, 124.1)
- added R7: 10k, Resistor_SMD:R_0805_2012Metric_Pad1.20x1.40mm_HandSolder, F.Cu at (99.0, 127.0)
- added R8: 10k, Resistor_SMD:R_0805_2012Metric_Pad1.20x1.40mm_HandSolder, F.Cu at (99.0, 130.0)
- added SW1: RECSW, Rotary_Encoder:RotaryEncoder_Alps_EC12E-Switch_Vertical_H20mm, F.Cu at (190.5, 91.1)
- A1: moved to B.Cu
- J1: footprint Connector_PinSocket_2.54mm:PinSocket_1x03_P2.54mm_Horizontal -> FSLP:Pololu FSLP 100
- moved FB2 150.6 mm to (125.0, 87.2), turned to -90 degrees
- moved C4 136.3 mm to (63.7, 35.1), turned to 90 degrees
- moved C5 133.6 mm to (66.2, 35.1), turned to 90 degrees
- moved C6 131.0 mm to (68.7, 35.1), turned to 90 degrees
- moved C7 128.4 mm to (71.2, 35.1), turned to 90 degrees
- moved C2 123.9 mm to (76.7, 34.3), turned to 90 degrees
- moved C3 120.7 mm to (80.0, 34.3), turned to 90 degrees
- moved R2 83.8 mm to (72.3, 39.2), turned to 90 degrees
- moved R3 81.2 mm to (75.3, 39.2), turned to 90 degrees
- moved C1 78.7 mm to (78.0, 39.4), turned to 90 degrees
- moved J1 70.8 mm to (66.0, 109.2), turned to -90 degrees
- moved R1 63.8 mm to (105.5, 129.5), turned to 90 degrees
- moved A1 42.6 mm to (99.6, 91.4), turned to 90 degrees
- moved U1 14.7 mm to (170.2, 83.8), turned to 180 degrees
Connections:
- A1 pad 5: /D2 -> /CLK
Other:
- board outline added: 141 x 48 mm

Commit message: Add files via upload
Parts:
- added C8: 47n DNI, Capacitor_SMD:C_0603_1608Metric_Pad1.08x0.95mm_HandSolder, F.Cu at (71.2, 134.5)
- added C9: 47n DNI, Capacitor_SMD:C_0603_1608Metric_Pad1.08x0.95mm_HandSolder, F.Cu at (71.2, 137.0)
- added J2: SJ-63063B, SJ63063B:CUI_SJ-63063B, B.Cu at (68.3, 101.0)
- added R9: Volume, PTV09A:PTV09A-4025F-B103, F.Cu at (112.0, 93.0)
- moved FB2 24.0 mm to (149.0, 86.5)
- moved R4 22.1 mm to (140.5, 77.3)
- moved R5 10.8 mm to (140.5, 92.8)
- moved J1 5.28 mm to (66.0, 114.5)
Other:
- board size 141 x 48 mm -> 141 x 53 mm

Commit message: Add files via upload
Parts:
- removed R9: Volume, PTV09A:PTV09A-4025F-B103
- added C10: 47n, Capacitor_SMD:C_0603_1608Metric_Pad1.08x0.95mm_HandSolder, F.Cu at (102.0, 97.0)
- added C11: 220u, Capacitor_SMD:C_1206_3216Metric_Pad1.33x1.80mm_HandSolder, F.Cu at (98.0, 96.0)
- added C12: 10u, Capacitor_SMD:C_1206_3216Metric_Pad1.33x1.80mm_HandSolder, F.Cu at (114.0, 103.0)
- added C13: 47u, Capacitor_SMD:C_1206_3216Metric_Pad1.33x1.80mm_HandSolder, F.Cu at (108.0, 103.0)
- added C14: 10u, Capacitor_SMD:C_1206_3216Metric_Pad1.33x1.80mm_HandSolder, F.Cu at (98.0, 88.0)
- added C15: 1n, Capacitor_SMD:C_0603_1608Metric_Pad1.08x0.95mm_HandSolder, F.Cu at (108.0, 89.0)
- added R10: 10K, PTV09A:PTV09A-4025F-B103, F.Cu at (116.0, 77.0)
- added R11: 10, Resistor_SMD:R_0805_2012Metric_Pad1.20x1.40mm_HandSolder, F.Cu at (98.0, 99.0)
- added U2: LM386, Package_DIP:DIP-8_W7.62mm, F.Cu at (114.8, 92.2)
- C2, C4, C5, FB2: moved to B.Cu
- moved C8 127.3 mm to (192.9, 97.0)
- moved C9 127.3 mm to (192.9, 99.5)
- moved C4 123.9 mm to (168.5, 101.1), turned to -90 degrees
- moved C5 123.9 mm to (171.0, 101.1), turned to -90 degrees
- moved C2 110.3 mm to (164.0, 101.7), turned to -90 degrees
- moved R6 93.0 mm to (188.0, 97.0)
- moved R7 93.0 mm to (188.0, 100.0)
- moved R8 93.0 mm to (188.0, 103.0)
- moved R1 48.6 mm to (82.0, 87.0), turned to -90 degrees
- moved C1 47.9 mm to (74.0, 87.1)
- moved R2 47.9 mm to (68.3, 86.9)
- moved R3 47.9 mm to (71.3, 86.9)
- moved C6 45.7 mm to (97.0, 71.0)
- moved C7 43.0 mm to (95.0, 71.0)
- moved C3 38.6 mm to (92.0, 71.0)
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Other:
- board size 141 x 53 mm -> 141 x 62 mm
