File: PCB/Synth_arduino_nano.kicad_sch (KiCad schematic)
At the start: 17 parts, among them J1 FSLP, J3 Encoder, U1 DM-OLED096-636

Commit message: Add files via upload
Parts:
- removed J3: Encoder, Connector_PinSocket_2.54mm:PinSocket_1x05_P2.54mm_Horizontal, symbol Connector:Conn_01x05_Socket
- added R6, R7, R8: 10k, Resistor_SMD:R_0805_2012Metric_Pad1.20x1.40mm_HandSolder, symbol Device:R
- added SW1: RECSW, Rotary_Encoder:RotaryEncoder_Alps_EC12E-Switch_Vertical_H20mm, symbol Device:RotaryEncoder_Switch
Connections:
- net +5V: now also R6.2, R7.2, R8.2
- net D3: now also R7.1, SW1.B
- net D8: now also R8.1, SW1.S1
- net GND: now also SW1.C, SW1.S2
- net D2 renamed CLK
- net CLK: now also R6.1, SW1.A
Other:
- note removed: "+"
- note removed: "CLK"
- note removed: "DT"
- note removed: "GND"
- note removed: "SW"

Commit message: Add files via upload
Parts:
- added C8, C9: 47n DNI, Capacitor_SMD:C_0603_1608Metric_Pad1.08x0.95mm_HandSolder, symbol Device:C
- added J2: SJ-63063B, SJ63063B:CUI_SJ-63063B, symbol SJ63063B:SJ-63063B
- added R9: Volume, PTV09A:PTV09A-4025F-B103, symbol PTV09A:PTV09A-4025F-B103
Connections:
- net AUDIO_OUT: now also R9.3
- net CLK: now also C8.1
- net D3: now also C9.1
- net GND: now also C8.2, C9.2, J2.1, R9.1
- new net: J2.2, R9.2
Other:
- moved on the sheet: A1, C1, C2, C3, C4, C5, C6, C7, FB2, J1, R1, R2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

Commit message: Add files via upload
Parts:
- removed R9: Volume, PTV09A:PTV09A-4025F-B103, symbol PTV09A:PTV09A-4025F-B103
- added C10: 47n, Capacitor_SMD:C_0603_1608Metric_Pad1.08x0.95mm_HandSolder, symbol Device:C
- added C11: 220u, Capacitor_SMD:C_1206_3216Metric_Pad1.33x1.80mm_HandSolder, symbol Device:C
- added C12, C14: 10u, Capacitor_SMD:C_1206_3216Metric_Pad1.33x1.80mm_HandSolder, symbol Device:C
- added C13: 47u, Capacitor_SMD:C_1206_3216Metric_Pad1.33x1.80mm_HandSolder, symbol Device:C
- added C15: 1n, Capacitor_SMD:C_0603_1608Metric_Pad1.08x0.95mm_HandSolder, symbol Device:C
- added R10: 10K, PTV09A:PTV09A-4025F-B103, symbol PTV09A:PTV09A-4025F-B103
- added R11: 10, Resistor_SMD:R_0805_2012Metric_Pad1.20x1.40mm_HandSolder, symbol Device:R
- added U2: LM386, Package_DIP:DIP-8_W7.62mm, symbol Amplifier_Audio:LM386
Connections:
- net +5V: now also C13.2, U2.6 (V+)
- net AUDIO_OUT: now also C14.1
- net GND: now also C12.2, C13.1, C15.2, R10.1, R11.1, U2.2 (-), U2.4 (GND)
- net at J2.2: now also C11.2
- new net: C15.1, R10.2, U2.3 (+)
- new net: C14.2, R10.3
- new net: C10.1, C11.1, U2.5
- new net: C10.2, R11.2
- new net: C12.1, U2.7 (BYPASS)
Other:
- moved on the sheet: C1, J2, R2, R3

Commit message: Add files via upload
Parts:
- added C16: DNI, Capacitor_SMD:C_0603_1608Metric_Pad1.08x0.95mm_HandSolder, symbol Device:C
- added R9: 0, Resistor_SMD:R_0805_2012Metric_Pad1.20x1.40mm_HandSolder, symbol Device:R
Connections:
- net AUDIO_OUT: now also R3.1, R9.2; no longer C14.1
- net GND: now also C16.2; no longer R3.1
- new net: C14.1, C16.1, R9.1
Other:
- moved on the sheet: C1
